File: interface.kicad_pcb (KiCad board)
At the start: 2 copper layers, 36.8 x 66 mm, 35 parts, among them U1 THERMAL, U2 SX1308

Commit message: add note
Parts:
- moved ? 1.87 mm to (138.6, 60.2)
- moved ? 1.60 mm to (128.1, 60.5)
Other:
- board text added: "+5V"
- board text added: "D0"
- board text added: "D1"
- board text added: "D10"
- board text added: "D11"
- board text added: "D12"
- board text added: "D13"
- board text added: "D14"
- board text added: "D15"
- board text added: "D2"
- board text added: "D3"
- board text added: "D4"
- board text added: "D5"
- board text added: "D6"
- board text added: "D7"
- board text added: "D8"
- board text added: "D9"
- board text added: "GND"
- board text added: "HSYN"
- board text added: "PCLK"
- board text added: "PEN"
- board text added: "RX"
- board text added: "TX"
- board text added: "VSYN"
Changed lines of the file:
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@@
     (area 124.384999 53.635 161.365001 120.725001)
     (thickness 1.6)
-    (drawings 5)
+    (drawings 29)
     (tracks 251)
     (zones 0)
@@
   (module pin24:pin24 (layer F.Cu)
     (at 154.94 55.88)
-    (fp_text reference J1 (at -1.27 1.27) (layer F.SilkS)
+    (fp_text reference J1 (at -2.34 0.62) (layer F.SilkS)
       (effects (font (size 1 1) (thickness 0.15)))
     )
@@
   )
   (module Symbols:WEEE-Logo_4.2x6mm_SilkScreen (layer F.Cu)
-    (at 128.1 58.9)
+    (at 128.1 60.5)
     (descr "Waste Electrical and Electronic Equipment Directive")
     (tags "Logo WEEE")
@@
   )
   (module Symbols:KiCad-Logo_6mm_SilkScreen (layer F.Cu)
-    (at 139.1 58.4)
+    (at 138.6 60.2)
     (descr "KiCad Logo")
     (tags "Logo KiCad")
@@
       (xy -3.046536 -2.947564) (xy -2.941012 -2.973419) (xy -2.833142 -2.978732) (xy -2.726079 -2.96351)) (layer F.SilkS) (width 0.01))
   )
-  (gr_text "Thermal\nCamera" (at 131.5 64.7) (layer F.Cu)
+  (gr_text D10 (at 153 88.8) (layer F.SilkS)
+    (effects (font (size 1 1) (thickness 0.2)))
+  )
+  (gr_text D9 (at 152.6 86.3) (layer F.SilkS)
+    (effects (font (size 1 1) (thickness 0.2)))
+  )
+  (gr_text D8 (at 152.6 83.8) (layer F.SilkS)
+    (effects (font (size 1 1) (thickness 0.2)))
+  )
+  (gr_text D7 (at 152.6 81.2) (layer F.SilkS)
+    (effects (font (size 1 1) (thickness 0.2)))
+  )
+  (gr_text D6 (at 152.7 78.6) (layer F.SilkS)
+    (effects (font (size 1 1) (thickness 0.2)))
+  )
+  (gr_text D5 (at 152.6 76.2) (layer F.SilkS)
+    (effects (font (size 1 1) (thickness 0.2)))
+  )
+  (gr_text D4 (at 152.7 73.6) (layer F.SilkS)
+    (effects (font (size 1 1) (thickness 0.2)))
+  )
+  (gr_text D3 (at 152.7 71.1) (layer F.SilkS)
+    (effects (font (size 1 1) (thickness 0.2)))
+  )
+  (gr_text D2 (at 152.7 68.5) (layer F.SilkS)
+    (effects (font (size 1 1) (thickness 0.2)))
+  )
+  (gr_text D1 (at 152.7 65.8) (layer F.SilkS)
+    (effects (font (size 1 1) (thickness 0.2)))
+  )
+  (gr_text D0 (at 152.7 63.4) (layer F.SilkS)
+    (effects (font (size 1 1) (thickness 0.2)))
+  )
+  (gr_text VSYN (at 152.4 60.8) (layer F.SilkS)
+    (effects (font (size 1 1) (thickness 0.2)))
+  )
+  (gr_text HSYN (at 152.5 58.6) (layer F.SilkS)
+    (effects (font (size 1 1) (thickness 0.2)))
+  )
+  (gr_text D11 (at 153 91.4) (layer F.SilkS)
+    (effects (font (size 1 1) (thickness 0.2)))
+  )
+  (gr_text D12 (at 153 94) (layer F.SilkS)
+    (effects (font (size 1 1) (thickness 0.2)))
+  )
+  (gr_text D13 (at 153.1 96.5) (layer F.SilkS)
+    (effects (font (size 1 1) (thickness 0.2)))
+  )
+  (gr_text D14 (at 153.1 99.1) (layer F.SilkS)
+    (effects (font (size 1 1) (thickness 0.2)))
+  )
+  (gr_text D15 (at 153.1 101.6) (layer F.SilkS)
+    (effects (font (size 1 1) (thickness 0.2)))
+  )
+  (gr_text PCLK (at 152.9 104.1) (layer F.SilkS)
+    (effects (font (size 1 1) (thickness 0.2)))
+  )
+  (gr_text TX (at 153.2 106.7) (layer F.SilkS)
+    (effects (font (size 1 1) (thickness 0.2)))
+  )
+  (gr_text RX (at 153.3 109.2) (layer F.SilkS)
+    (effects (font (size 1 1) (thickness 0.2)))
+  )
+  (gr_text PEN (at 152.9 111.8) (layer F.SilkS)
+    (effects (font (size 1 1) (thickness 0.2)))
+  )
+  (gr_text +5V (at 152.7 114.3) (layer F.SilkS)
+    (effects (font (size 1 1) (thickness 0.2)))
+  )
+  (gr_text GND (at 152.9 117.1) (layer F.SilkS)
+    (effects (font (size 1 1) (thickness 0.2)))
+  )
+  (gr_text "Thermal\nCamera" (at 132.1 66.4) (layer F.Cu)
     (effects (font (size 1.5 1.5) (thickness 0.3)))
   )

Commit message: finish and factory
Routing:
- added copper zone on B.Cu, net GND
- added copper zone on F.Cu, net GND
Changed lines of the file:
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@@
     (trace_clearance 0.15)
     (zone_clearance 0.508)
-    (zone_45_only no)
+    (zone_45_only yes)
     (trace_min 0.2)
     (segment_width 0.2)
@@
   (segment (start 141.6 80.6) (end 141.6 75) (width 0.25) (layer F.Cu) (net 52))
   (segment (start 139.4 82.8) (end 141.6 80.6) (width 0.25) (layer F.Cu) (net 52))
+  (zone (net 0) (net_name "") (layer F.Cu) (hatch edge 0.508)
+    (connect_pads (clearance 0.508))
+    (min_thickness 0.254)
+    (keepout (tracks allowed) (vias allowed) (copperpour not_allowed))
+    (fill (arc_segments 16) (thermal_gap 0.508) (thermal_bridge_width 0.508))
+    (polygon
+      (pts
+        (xy 143.9 104.8) (xy 139.5 104.8) (xy 139.5 103.4) (xy 143.9 103.4)
+      )
+    )
+  )
+  (zone (net 0) (net_name "") (layer F.Cu) (hatch edge 0.508)
+    (connect_pads (clearance 0.508))
+    (min_thickness 0.254)
+    (keepout (tracks allowed) (vias allowed) (copperpour not_allowed))
+    (fill (arc_segments 16) (thermal_gap 0.508) (thermal_bridge_width 0.508))
+    (polygon
+      (pts
+        (xy 147 113.8) (xy 150.2 113.8) (xy 150.2 117.3) (xy 146.9 117.3) (xy 146.9 113.8)
+      )
+    )
+  )
+  (zone (net 0) (net_name "") (layer F.Cu) (hatch edge 0.508)
+    (connect_pads (clearance 0.508))
+    (min_thickness 0.254)
+    (keepout (tracks allowed) (vias allowed) (copperpour not_allowed))
+    (fill (arc_segments 16) (thermal_gap 0.508) (thermal_bridge_width 0.508))
+    (polygon
+      (pts
+        (xy 130.4 73.7) (xy 131.2 74.5) (xy 127.8 77.9) (xy 127.8 99.2) (xy 131.2 99.2)
+        (xy 131.2 103.1) (xy 129.1 103.1) (xy 129.1 102.9) (xy 127.8 100.368421) (xy 127.8 102.2)
+        (xy 128.3 102.2) (xy 129 102.9) (xy 129 110.9) (xy 130.2 112.1) (xy 130.2 114.8)
+        (xy 128.6 114.8) (xy 127.9 114.1) (xy 126.6 114.1) (xy 125.7 113.2) (xy 125.7 103.2)
+        (xy 126.6 102.3) (xy 126.4 102.3) (xy 126.4 77.2) (xy 130.2 73.4) (xy 130.4 73.4)
+      )
+    )
+  )
+  (zone (net 0) (net_name "") (layer F.Cu) (hatch edge 0.508)
+    (connect_pads (clearance 0.508))
+    (min_thickness 0.254)
+    (keepout (tracks allowed) (vias allowed) (copperpour not_allowed))
+    (fill (arc_segments 16) (thermal_gap 0.508) (thermal_bridge_width 0.508))
+    (polygon
+      (pts
+        (xy 134.5 103.1) (xy 132.3 103.1) (xy 132.3 99.9) (xy 134.5 99.9)
+      )
+    )
+  )
+  (zone (net 2) (net_name GND) (layer F.Cu) (hatch edge 0.508)
+    (connect_pads (clearance 0.508))
+    (min_thickness 0.254)
+    (fill yes (arc_segments 16) (thermal_gap 0.508) (thermal_bridge_width 0.508))
+    (polygon
+      (pts
+        (xy 161.3 120.6) (xy 124.5 120.6) (xy 124.5 54.6) (xy 161.3 54.6)
+      )
+    )
+  )
+  (zone (net 2) (net_name GND) (layer B.Cu) (hatch edge 0.508)
+    (connect_pads (clearance 0.508))
+    (min_thickness 0.254)
+    (fill yes (arc_segments 16) (thermal_gap 0.508) (thermal_bridge_width 0.508))
+    (polygon
+      (pts
+        (xy 161.3 120.6) (xy 124.5 120.6) (xy 124.5 54.6) (xy 161.3 54.6)
+      )
+    )
+  )
 )
